Commit message: Refined wheel orientation, joystick behavior, and removed deprecated packages

File: src/mecca_description/urdf/meccabot.xacro (robot description, xacro)
@@ -1,245 +1,116 @@
 <?xml version="1.0"?>
 <robot xmlns:xacro="http://ros.org/wiki/xacro" name="meccabot_robot">
-    <xacro:include filename="inertial_macros.xacro"/>
-    <xacro:include filename="gazebo_control.xacro"/>
-    <xacro:property name="wheel_separation" value="0.3"/>
-    <!--=== Wheel and chassis dimensions ===-->
-    <xacro:property name="wheel_radius"    value="0.05"/>      <!-- 50 mm wheel radius -->
-    <xacro:property name="wheel_thickness" value="0.03"/>      <!-- 30 mm wheel thickness -->
-    <xacro:property name="chassis_length"  value="0.275"/>     <!-- 275 mm chassis length -->
-    <xacro:property name="chassis_width"   value="0.145"/>     <!-- 145 mm chassis width -->
-    <xacro:property name="chassis_height"  value="0.125"/>     <!-- 125 mm chassis height -->
-    <!--=== Key positioning parameters ===-->
-    <!-- Distance from robot center to chassis corners -->
-    <xacro:property name="chassis_half_length" value="${chassis_length/2}"/>
-    <xacro:property name="chassis_half_width" value="${chassis_width/2}"/>
-    <!-- Ground clearance: distance from ground to bottom of chassis -->
-    <xacro:property name="ground_clearance" value="0.015"/>    <!-- 15 mm clearance -->
-    <!-- Wheel offsets from chassis edges -->
-    <xacro:property name="wheel_x_offset"  value="0.05"/>      <!-- 50 mm from front/rear edges -->
-    <xacro:property name="wheel_y_offset"  value="0.0"/>       <!-- 0 mm from side edges (wheels aligned with chassis sides) -->
-    <!-- Z height for chassis origin from ground -->
-    <xacro:property name="chassis_z_offset" value="${wheel_radius + ground_clearance}"/>
-    <!-- Z offset for wheel centers relative to chassis_link -->
-    <xacro:property name="wheel_z_offset" value="${-ground_clearance}"/>
-    <!-- Define Colors -->
-    <material name="white">
-        <color rgba="1 1 1 1" />
-    </material>
-    <material name="orange">
-        <color rgba="1 0.3 0.1 1" />
-    </material>
-    <material name="red">
-        <color rgba="1 0 0 1" />
-    </material>
-    <material name="blue">
-        <color rgba="0.0 0.0 0.8 1.0" />
-    </material>
-    <material name="green">
-        <color rgba="0.2 0.9 0.2 1"/>
-    </material>
-    <material name="darkgrey">
-        <color rgba="0.1 0.1 0.1 1.0" />
-    </material>
-    <material name="grey">
-        <color rgba="0.5 0.5 0.5 1.0" />
-    </material>
-    <material name="black">
-        <color rgba="0 0 0 1" />
-    </material>
-    <!-- Base Link (Root) -->
-    <link name="base_link">
-        <!-- Add inertia to base_link to avoid TF errors -->
-        <inertial>
-            <origin xyz="0 0 0" rpy="0 0 0"/>
-            <mass value="0.1"/>
-            <inertia ixx="0.001" ixy="0.0" ixz="0.0" iyy="0.001" iyz="0.0" izz="0.001"/>
-        </inertial>
-    </link>
-    <!-- Fixed joint from base_link → chassis_link -->
-<joint name="base_to_chassis" type="fixed">
+  <xacro:include filename="inertial_macros.xacro"/>
+  <xacro:include filename="gazebo_control.xacro"/>
+  <!-- Parameters -->
+  <xacro:property name="wheel_radius" value="0.05"/>
+  <xacro:property name="wheel_thickness" value="0.03"/>
+  <xacro:property name="chassis_length" value="0.275"/>
+  <xacro:property name="chassis_width" value="0.145"/>
+  <xacro:property name="chassis_height" value="0.125"/>
+  <xacro:property name="ground_clearance" value="0.015"/>
+  <xacro:property name="chassis_half_length" value="${chassis_length/2}"/>
+  <xacro:property name="chassis_half_width" value="${chassis_width/2}"/>
+  <xacro:property name="wheel_x_offset" value="0.05"/>
+  <xacro:property name="wheel_y_offset" value="0.0"/>
+  <xacro:property name="chassis_z_offset" value="${wheel_radius + ground_clearance}"/>
+  <xacro:property name="wheel_z_offset" value="${-ground_clearance}"/>
+  <!-- Colors -->
+  <material name="grey"><color rgba="0.5 0.5 0.5 1.0"/></material>
+  <material name="green"><color rgba="0.2 0.9 0.2 1.0"/></material>
+  <!-- Base link -->
+  <link name="base_link">
+    <inertial>
+      <origin xyz="0 0 0" rpy="0 0 0"/>
+      <mass value="0.1"/>
+      <inertia ixx="0.001" ixy="0.0" ixz="0.0" iyy="0.001" iyz="0.0" izz="0.001"/>
+    </inertial>
+  </link>
+  <joint name="base_to_chassis" type="fixed">
     <parent link="base_link"/>
-    <child  link="chassis_link"/>
-    <!-- Raise chassis so it has proper ground clearance -->
+    <child link="chassis_link"/>
     <origin xyz="0 0 ${chassis_z_offset}" rpy="0 0 0"/>
   </joint>
-  <!-- Simplified chassis as a box 0.275 × 0.145 × 0.125 m -->
+  <!-- Chassis -->
   <link name="chassis_link">
-    <!-- Inertial: box centered above the ground plane -->
     <inertial>
-      <!-- place COM at half the height above ground -->
       <origin xyz="0 0 0.0625" rpy="0 0 0"/>
       <mass value="5.0"/>
       <inertia
-        ixx="${(1/12)*5.0*(0.145*0.145 + 0.125*0.125)}"
+        ixx="${(1/12)*5.0*(chassis_width*chassis_width + chassis_height*chassis_height)}"
         ixy="0.0" ixz="0.0"
-        iyy="${(1/12)*5.0*(0.275*0.275 + 0.125*0.125)}"
+        iyy="${(1/12)*5.0*(chassis_length*chassis_length + chassis_height*chassis_height)}"
         iyz="0.0"
-        izz="${(1/12)*5.0*(0.275*0.275 + 0.145*0.145)}"/>
+        izz="${(1/12)*5.0*(chassis_length*chassis_length + chassis_width*chassis_width)}"/>
     </inertial>
-    <!-- Visual -->
     <visual>
-      <!-- box’s center at COM -->
       <origin xyz="0 0 0.0625" rpy="0 0 0"/>
       <geometry>
-        <box size="0.275 0.145 0.125"/>
+        <box size="${chassis_length} ${chassis_width} ${chassis_height}"/>
       </geometry>
       <material name="green"/>
     </visual>
-    <!-- Collision: same as visual -->
     <collision>
       <origin xyz="0 0 0.0625" rpy="0 0 0"/>
       <geometry>
-        <box size="0.275 0.145 0.125"/>
+        <box size="${chassis_length} ${chassis_width} ${chassis_height}"/>
       </geometry>
     </collision>
   </link>
-<gazebo reference="chassis_link">
-        <material>Gazebo/Green</material>
-    </gazebo>
-  <!-- Wheels           -->
-  <!-- Front Left Wheel -->
-  <joint name="front_left_wheel_joint" type="continuous">
-    <parent link="chassis_link"/>
-    <child  link="front_left_wheel"/>
-    <origin xyz="${chassis_half_length - wheel_x_offset}
-               ${chassis_half_width + wheel_thickness/2}
-               ${wheel_z_offset}" rpy="0 0 0"/>
-    <axis   xyz="0 1 0"/>
-  </joint>
-    <link name="front_left_wheel">
-    <inertial>
+  <!-- Wheel macro -->
+  <xacro:macro name="wheel" params="name x y z rpy">
+    <joint name="${name}_joint" type="continuous">
+      <parent link="chassis_link"/>
+      <child link="${name}"/>
+      <origin xyz="${x} ${y} ${z}" rpy="${rpy}"/>
+      <axis xyz="0 1 0"/>
+    </joint>
+    <link name="${name}">
+      <inertial>
         <origin xyz="0 0 0" rpy="0 0 0"/>
         <mass value="0.5"/>
         <inertia
-            ixx="${(1/12) * 0.5 * (3*wheel_radius*wheel_radius + wheel_thickness*wheel_thickness)}"
-            ixy="0.0" ixz="0.0"
-            iyy="${(1/12) * 0.5 * (3*wheel_radius*wheel_radius + wheel_thickness*wheel_thickness)}"
-            iyz="0.0"
-            izz="${(1/2) * 0.5 * wheel_radius*wheel_radius}"/>
-    </inertial>
-    <visual>
-        <origin xyz="0 0 0" rpy="0 0 1.5708"/>
+          ixx="0.001" ixy="0.0" ixz="0.0"
+          iyy="0.001" iyz="0.0"
+          izz="0.001"/>
+      </inertial>
+      <visual>
+        <origin xyz="0 0 0" rpy="0 1.5708 0"/>
         <geometry>
-            <mesh filename="package://mecca_description/meshes/fl_wheel_link.stl" scale="1 1 1"/>
+          <cylinder radius="${wheel_radius}" length="${wheel_thickness}"/>
         </geometry>
         <material name="grey"/>
-    </visual>
-    <collision>
-        <origin xyz="0 0 0" rpy="0 0 1.5708"/>
+      </visual>
+      <collision>
+        <origin xyz="0 0 0" rpy="0 1.5708" 0/>
         <geometry>
-            <mesh filename="package://mecca_description/meshes/fl_wheel_link.stl" scale="1 1 1"/>
+          <cylinder radius="${wheel_radius}" length="${wheel_thickness}"/>
         </geometry>
-    </collision>
+      </collision>
     </link>
-  <!-- Front Right Wheel -->
-  <joint name="front_right_wheel_joint" type="continuous">
-    <parent link="chassis_link"/>
-    <child  link="front_right_wheel"/>
-    <origin xyz="${chassis_half_length - wheel_x_offset}
-               ${-(chassis_half_width + wheel_thickness/2)}
-               ${wheel_z_offset}" rpy="0 0 0"/>
-    <axis   xyz="0 1 0"/>
-  </joint>
-    <link name="front_right_wheel">
-    <inertial>
-        <origin xyz="0 0 0" rpy="0 0 0"/>
-        <mass value="0.5"/>
-        <inertia
-            ixx="${(1/12) * 0.5 * (3*wheel_radius*wheel_radius + wheel_thickness*wheel_thickness)}"
-            ixy="0.0" ixz="0.0"
-            iyy="${(1/12) * 0.5 * (3*wheel_radius*wheel_radius + wheel_thickness*wheel_thickness)}"
-            iyz="0.0"
-            izz="${(1/2) * 0.5 * wheel_radius*wheel_radius}"/>
-    </inertial>
-    <visual>
-        <origin xyz="0 0 0" rpy="0 0 -1.5708"/>
-        <geometry>
-            <mesh filename="package://mecca_description/meshes/fr_wheel_link.stl" scale="1 1 1"/>
-        </geometry>
-        <material name="grey"/>
-    </visual>
-    <collision>
-        <origin xyz="0 0 0" rpy="0 0 -1.5708"/>
-        <geometry>
-            <mesh filename="package://mecca_description/meshes/fr_wheel_link.stl" scale="1 1 1"/>
-        </geometry>
-    </collision>
-    </link>
-  <!-- Rear Left Wheel -->
-  <joint name="rear_left_wheel_joint" type="continuous">
-    <parent link="chassis_link"/>
-    <child  link="rear_left_wheel"/>
-    <origin xyz="${-(chassis_half_length - wheel_x_offset)}
-               ${chassis_half_width + wheel_thickness/2}
-               ${wheel_z_offset}" rpy="0 0 0"/>
-    <axis   xyz="0 1 0"/>
-  </joint>
-    <link name="rear_left_wheel">
-    <inertial>
-        <origin xyz="0 0 0" rpy="0 0 0"/>
-        <mass value="0.5"/>
-        <inertia
-            ixx="${(1/12) * 0.5 * (3*wheel_radius*wheel_radius + wheel_thickness*wheel_thickness)}"
-            ixy="0.0" ixz="0.0"
-            iyy="${(1/12) * 0.5 * (3*wheel_radius*wheel_radius + wheel_thickness*wheel_thickness)}"
-            iyz="0.0"
-            izz="${(1/2) * 0.5 * wheel_radius*wheel_radius}"/>
-    </inertial>
-    <visual>
-        <origin xyz="0 0 0" rpy="0 0 1.5708"/>
-        <geometry>
-            <mesh filename="package://mecca_description/meshes/rl_wheel_link.stl" scale="1 1 1"/>
-        </geometry>
-        <material name="grey"/>
-    </visual>
-    <collision>
-         <origin xyz="0 0 0" rpy="0 0 1.5708"/>
-         <geometry>
-            <mesh filename="package://mecca_description/meshes/rl_wheel_link.stl" scale="1 1 1"/>
-        </geometry>
-    </collision>
-    </link>
-  <!-- Rear Right Wheel -->
-  <joint name="rear_right_wheel_joint" type="continuous">
-    <parent link="chassis_link"/>
-    <child  link="rear_right_wheel"/>
-    <origin xyz="${-(chassis_half_length - wheel_x_offset)}
-               ${-(chassis_half_width + wheel_thickness/2)}
-               ${wheel_z_offset}" rpy="0 0 0"/>
-    <axis   xyz="0 1 0"/>
-  </joint>
-    <link name="rear_right_wheel">
-    <inertial>
-        <origin xyz="0 0 0" rpy="0 0 0"/>
-        <mass value="0.5"/>
-        <inertia
-            ixx="${(1/12) * 0.5 * (3*wheel_radius*wheel_radius + wheel_thickness*wheel_thickness)}"
-            ixy="0.0" ixz="0.0"
-            iyy="${(1/12) * 0.5 * (3*wheel_radius*wheel_radius + wheel_thickness*wheel_thickness)}"
-            iyz="0.0"
-            izz="${(1/2) * 0.5 * wheel_radius*wheel_radius}"/>
-    </inertial>
-    <visual>
-        <origin xyz="0 0 0" rpy="0 0 -1.5708"/>
-        <geometry>
-            <mesh filename="package://mecca_description/meshes/rr_wheel_link.stl" scale="1 1 1"/>
-        </geometry>
-        <material name="grey"/>
-    </visual>
-    <collision>
-        <origin xyz="0 0 0" rpy="0 0 -1.5708"/>
-        <geometry>
-            <mesh filename="package://mecca_description/meshes/rr_wheel_link.stl" scale="1 1 1"/>
-        </geometry>
-    </collision>
-    </link>
-  <!-- Lidar Mount -->
+  </xacro:macro>
+  <!-- Instantiate wheels -->
+  <xacro:wheel name="front_left_wheel"
+               x="${chassis_half_length - wheel_x_offset}"
+               y="${chassis_half_width + wheel_thickness/2}"
+               z="${wheel_z_offset}"
+               rpy="0 0 0"/>
+  <xacro:wheel name="front_right_wheel"
+               x="${chassis_half_length - wheel_x_offset}"
+               y="${-(chassis_half_width + wheel_thickness/2)}"
+               z="${wheel_z_offset}"
+               rpy="0 0 0"/>
+  <xacro:wheel name="rear_left_wheel"
+               x="${-(chassis_half_length - wheel_x_offset)}"
+               y="${chassis_half_width + wheel_thickness/2}"
+               z="${wheel_z_offset}"
+               rpy="0 0 0"/>
+  <xacro:wheel name="rear_right_wheel"
+               x="${-(chassis_half_length - wheel_x_offset)}"
+               y="${-(chassis_half_width + wheel_thickness/2)}"
+               z="${wheel_z_offset}"
+               rpy="0 0 0"/>
+  <!-- Lidar -->
   <link name="lidar_mount">
-    <inertial>
-      <origin xyz="0 0 0" rpy="0 0 0"/>
-      <mass value="0.2"/>
-      <inertia ixx="0.0001" ixy="0.0" ixz="0.0" iyy="0.0001" iyz="0.0" izz="0.0001"/>
-    </inertial>
     <visual>
       <geometry>
@@ -259,25 +130,25 @@
     <origin xyz="-0.050 0 ${0.14 + chassis_z_offset}" rpy="0 0 0"/>
   </joint>
-  <!-- ROS2 Control Interface -->
+  <!-- ROS2 Control Interfaces -->
   <ros2_control name="MecanumRobot" type="system">
-      <hardware>
-          <plugin>mecanum_hardware_interface/MecanumHardware</plugin>
-      </hardware>
-      <joint name="front_left_wheel_joint">
-          <command_interface name="velocity"/>
-          <state_interface name="velocity"/>
-      </joint>
-      <joint name="front_right_wheel_joint">
-          <command_interface name="velocity"/>
-          <state_interface name="velocity"/>
-      </joint>
-      <joint name="rear_left_wheel_joint">
-          <command_interface name="velocity"/>
-          <state_interface name="velocity"/>
-      </joint>
-      <joint name="rear_right_wheel_joint">
-          <command_interface name="velocity"/>
-          <state_interface name="velocity"/>
-      </joint>
+    <hardware>
+      <plugin>mecanum_hardware_interface/MecanumHardware</plugin>
+    </hardware>
+    <joint name="front_left_wheel_joint">
+      <command_interface name="velocity"/>
+      <state_interface name="velocity"/>
+    </joint>
+    <joint name="front_right_wheel_joint">
+      <command_interface name="velocity"/>
+      <state_interface name="velocity"/>
+    </joint>
+    <joint name="rear_left_wheel_joint">
+      <command_interface name="velocity"/>
+      <state_interface name="velocity"/>
+    </joint>
+    <joint name="rear_right_wheel_joint">
+      <command_interface name="velocity"/>
+      <state_interface name="velocity"/>
+    </joint>
   </ros2_control>
 </robot>

Commit message: fixing wheel orientation.

File: src/mecca_description/urdf/meccabot.xacro (robot description, xacro)
@@ -76,5 +76,5 @@
       </inertial>
       <visual>
-        <origin xyz="0 0 0" rpy="0 1.5708 0"/>
+        <origin xyz="0 0 0" rpy="1.5708 0 0"/>
         <geometry>
           <cylinder radius="${wheel_radius}" length="${wheel_thickness}"/>
@@ -83,5 +83,5 @@
       </visual>
       <collision>
-        <origin xyz="0 0 0" rpy="0 1.5708" 0/>
+        <origin xyz="0 0 0" rpy="1.5708 0 0"/>
         <geometry>
           <cylinder radius="${wheel_radius}" length="${wheel_thickness}"/>

Commit message: Initial version of mecca_hardware_interface for ROS COntrol.

File: src/mecca_description/urdf/meccabot.xacro (robot description, xacro)
@@ -16,7 +16,29 @@
   <xacro:property name="chassis_z_offset" value="${wheel_radius + ground_clearance}"/>
   <xacro:property name="wheel_z_offset" value="${-ground_clearance}"/>
-  <!-- Colors -->
-  <material name="grey"><color rgba="0.5 0.5 0.5 1.0"/></material>
-  <material name="green"><color rgba="0.2 0.9 0.2 1.0"/></material>
+    <!-- Define Colors -->
+    <material name="white">
+        <color rgba="1 1 1 1" />
+    </material>
+    <material name="orange">
+        <color rgba="1 0.3 0.1 1" />
+    </material>
+    <material name="red">
+        <color rgba="1 0 0 1" />
+    </material>
+    <material name="blue">
+        <color rgba="0.0 0.0 0.8 1.0" />
+    </material>
+    <material name="green">
+        <color rgba="0.2 0.9 0.2 1"/>
+    </material>
+    <material name="darkgrey">
+        <color rgba="0.1 0.1 0.1 1.0" />
+    </material>
+    <material name="grey">
+        <color rgba="0.5 0.5 0.5 1.0" />
+    </material>
+    <material name="black">
+        <color rgba="0 0 0 1" />
+    </material>
   <!-- Base link -->
   <link name="base_link">
@@ -130,25 +152,28 @@
     <origin xyz="-0.050 0 ${0.14 + chassis_z_offset}" rpy="0 0 0"/>
   </joint>
-  <!-- ROS2 Control Interfaces -->
-  <ros2_control name="MecanumRobot" type="system">
-    <hardware>
-      <plugin>mecanum_hardware_interface/MecanumHardware</plugin>
-    </hardware>
-    <joint name="front_left_wheel_joint">
-      <command_interface name="velocity"/>
-      <state_interface name="velocity"/>
-    </joint>
-    <joint name="front_right_wheel_joint">
-      <command_interface name="velocity"/>
-      <state_interface name="velocity"/>
-    </joint>
-    <joint name="rear_left_wheel_joint">
-      <command_interface name="velocity"/>
-      <state_interface name="velocity"/>
-    </joint>
-    <joint name="rear_right_wheel_joint">
-      <command_interface name="velocity"/>
-      <state_interface name="velocity"/>
-    </joint>
-  </ros2_control>
+<ros2_control name="MecanumRobot" type="system">
+  <hardware>
+    <plugin>mecanum_hardware_interface/MecanumHardware</plugin>
+  </hardware>
+  <joint name="front_left_wheel_joint">
+    <command_interface name="velocity"/>
+    <state_interface name="position"/>
+    <state_interface name="velocity"/>
+  </joint>
+  <joint name="front_right_wheel_joint">
+    <command_interface name="velocity"/>
+    <state_interface name="position"/>
+    <state_interface name="velocity"/>
+  </joint>
+  <joint name="rear_left_wheel_joint">
+    <command_interface name="velocity"/>
+    <state_interface name="position"/>
+    <state_interface name="velocity"/>
+  </joint>
+  <joint name="rear_right_wheel_joint">
+    <command_interface name="velocity"/>
+    <state_interface name="position"/>
+    <state_interface name="velocity"/>
+  </joint>
+</ros2_control>
 </robot>
